File: kicad/usb2ftdi.kicad_pcb (KiCad board)
At the start: 2 copper layers, 35 x 22 mm, 11 parts, among them J1 USB-Micro, J2 USB-Mini, J3 USB-B, P1 CONN_1, P2 CONN_1

Commit message: complete, ready to order
Parts:
- removed P2: CONN_1, Connect:1pin
- C1: footprint Capacitors_ThroughHole:Capacitor3MMDiscRM2.5 -> usb2ftdi:C1
- H1: footprint Pin_Headers:Pin_Header_Angled_1x06 -> usb2ftdi:Socket_Strip_Angled_1x06; moved to B.Cu
- J1: footprint Connect:USB_Micro-B -> usb2ftdi:USB_B_Micro
- J2: footprint Connect:USB_Mini-B -> usb2ftdi:USB_Mini-B
- J3: footprint Connect:USB_B -> usb2ftdi:USB_B
- P1: footprint Connect:1pin -> usb2ftdi:Screw_3mm
- Z1: footprint Pin_Arrays:pin_array_1x01 -> usb2ftdi:Logo-WL3
- Z2: footprint Pin_Arrays:pin_array_1x01 -> usb2ftdi:Logo-WL3; moved to B.Cu
- Z3: footprint Pin_Arrays:pin_array_1x01 -> usb2ftdi:Logo_silk_OSHW_6x6mm; moved to B.Cu
- Z4: footprint Pin_Arrays:pin_array_1x01 -> usb2ftdi:Logo_silk_OSHW_6x6mm
- moved Z3 162.2 mm to (34.2, 27.8), turned to 270 degrees
- moved Z2 158.4 mm to (30.0, 33.5), turned to 270 degrees
- moved C1 140.5 mm to (41.0, 28.5)
- moved Z4 139.0 mm to (44.0, 40.0)
- moved J2 135.7 mm to (28.5, 30.0)
- moved J1 131.3 mm to (33.8, 40.0)
- moved P1 130.4 mm to (47.0, 28.0)
- moved H1 129.9 mm to (54.2, 34.5), turned to 90 degrees
- moved Z1 128.5 mm to (55.0, 36.0)
- moved J3 125.2 mm to (45.0, 39.0), turned to 180 degrees
Connections:
- J2 pad 2: Net-(J2-Pad2) -> (no net)
Routing:
- net GND: track 75.4 -> 98.1 mm
- net /V_USB: track 40.9 -> 33.1 mm
- added copper zone on B.Cu, net GND
Other:
- board size 35 x 22 mm -> 35 x 20 mm
- net class 0.5 added: clearance 0.254, trace_width 0.5, via_dia 0.889, via_drill 0.635
- net class 1.0 added: clearance 0.254, trace_width 1, via_dia 0.889, via_drill 0.635
- board text added: "wyolum.com"
