File: kicad/usb2ftdi.sch (KiCad schematic (older format))
At the start: 11 parts, among them J1 USB-Micro, J2 USB-Mini, J3 USB-B, P1 CONN_1, P2 CONN_1

Commit message: complete, ready to order
Parts:
- removed P2: CONN_1, Connect:1pin, symbol CONN_1
- C1: footprint Capacitors_ThroughHole:Capacitor3MMDiscRM2.5 -> usb2ftdi:C1
- H1: footprint Pin_Headers:Pin_Header_Angled_1x06 -> usb2ftdi:Socket_Strip_Angled_1x06
- J1: footprint Connect:USB_Micro-B -> usb2ftdi:USB_B_Micro
- J2: footprint Connect:USB_Mini-B -> usb2ftdi:USB_Mini-B
- J3: footprint Connect:USB_B -> usb2ftdi:USB_B
- P1: footprint Connect:1pin -> usb2ftdi:Screw_3mm
- Z1, Z2: footprint Pin_Arrays:pin_array_1x01 -> usb2ftdi:Logo-WL3
- Z3, Z4: footprint Pin_Arrays:pin_array_1x01 -> usb2ftdi:Logo_silk_OSHW_6x6mm
Connections:
- net GND: now also J1.10 (T5), J1.11 (T6)
- no-connect marks 14 -> 13
Changed lines of the file:
@@
 	4800 3050 5725 3050
-$Comp
-L CONN_1 P2
-U 1 1 54CD2E9C
-P 4975 6950
-F 0 "P2" V 5050 6950 40  0000 L CNN
-F 1 "CONN_1" H 4975 7005 30  0001 C CNN
-F 2 "Connect:1pin" H 4975 6950 60  0001 C CNN
-F 3 "" H 4975 6950 60  0001 C CNN
-	1    4975 6950
-	0    -1   -1   0
-$EndComp
 $Comp
 L CONN_1 P1
@@
 F 0 "P1" V 4850 6950 40  0000 L CNN
 F 1 "CONN_1" H 4775 7005 30  0001 C CNN
-F 2 "Connect:1pin" H 4775 6950 60  0001 C CNN
+F 2 "usb2ftdi:Screw_3mm" H 4775 6950 60  0001 C CNN
 F 3 "" H 4775 6950 60  0001 C CNN
 	1    4775 6950
@@
 F 0 "C1" H 4625 3225 50  0000 L CNN
 F 1 "100n" H 4625 3075 50  0000 L CNN
-F 2 "Capacitors_ThroughHole:Capacitor3MMDiscRM2.5" H 4525 3150 60  0001 C CNN
+F 2 "usb2ftdi:C1" H 4525 3150 60  0001 C CNN
 F 3 "" H 4525 3150 60  0001 C CNN
 	1    4525 3150
@@
 F 0 "H1" V 6025 3100 60  0000 C CNN
 F 1 "FTDI" V 6125 3100 60  0000 C CNN
-F 2 "Pin_Headers:Pin_Header_Angled_1x06" H 6075 3100 60  0001 C CNN
+F 2 "usb2ftdi:Socket_Strip_Angled_1x06" H 6075 3100 60  0001 C CNN
 F 3 "" H 6075 3100 60  0001 C CNN
 	1    6075 3100
@@
 MOUNT HOLES
 NoConn ~ 4775 7100
-NoConn ~ 4975 7100
 $Comp
 L SCREW Z3
@@
 F 0 "Z3" V 6025 6950 40  0000 L CNN
 F 1 "CONN_1" H 5950 7005 30  0001 C CNN
-F 2 "Pin_Arrays:pin_array_1x01" H 5950 6950 60  0001 C CNN
+F 2 "usb2ftdi:Logo_silk_OSHW_6x6mm" H 5950 6950 60  0001 C CNN
 F 3 "" H 5950 6950 60  0001 C CNN
 	1    5950 6950
@@
 F 0 "Z4" V 6225 6950 40  0000 L CNN
 F 1 "CONN_1" H 6150 7005 30  0001 C CNN
-F 2 "Pin_Arrays:pin_array_1x01" H 6150 6950 60  0001 C CNN
+F 2 "usb2ftdi:Logo_silk_OSHW_6x6mm" H 6150 6950 60  0001 C CNN
 F 3 "" H 6150 6950 60  0001 C CNN
 	1    6150 6950
@@
 F 0 "Z2" V 6025 6350 40  0000 L CNN
 F 1 "CONN_1" H 5950 6405 30  0001 C CNN
-F 2 "Pin_Arrays:pin_array_1x01" H 5950 6350 60  0001 C CNN
+F 2 "usb2ftdi:Logo-WL3" H 5950 6350 60  0001 C CNN
 F 3 "" H 5950 6350 60  0001 C CNN
 	1    5950 6350
@@
 F 0 "Z1" V 5825 6350 40  0000 L CNN
 F 1 "CONN_1" H 5750 6405 30  0001 C CNN
-F 2 "Pin_Arrays:pin_array_1x01" H 5750 6350 60  0001 C CNN
+F 2 "usb2ftdi:Logo-WL3" H 5750 6350 60  0001 C CNN
 F 3 "" H 5750 6350 60  0001 C CNN
 	1    5750 6350
@@
 F 0 "J1" H 925 1525 60  0000 C CNN
 F 1 "USB-Micro" H 775 1650 60  0000 C CNN
-F 2 "Connect:USB_Micro-B" H 1500 1600 60  0001 C CNN
+F 2 "usb2ftdi:USB_B_Micro" H 1500 1600 60  0001 C CNN
 F 3 "" H 1500 1600 60  0000 C CNN
 	1    1500 1600
@@
 F 0 "J2" H 925 3300 60  0000 C CNN
 F 1 "USB-Mini" H 775 3425 60  0000 C CNN
-F 2 "Connect:USB_Mini-B" H 1500 3375 60  0001 C CNN
+F 2 "usb2ftdi:USB_Mini-B" H 1500 3375 60  0001 C CNN
 F 3 "" H 1500 3375 60  0000 C CNN
 	1    1500 3375
@@
 F 0 "J3" H 925 5075 60  0000 C CNN
 F 1 "USB-B" H 775 5200 60  0000 C CNN
-F 2 "Connect:USB_B" H 1500 5150 60  0001 C CNN
+F 2 "usb2ftdi:USB_B" H 1500 5150 60  0001 C CNN
 F 3 "" H 1500 5150 60  0000 C CNN
 	1    1500 5150
@@
 Text Label 1850 5875 0    47   ~ 0
 GND
+Wire Wire Line
+	1200 1000 1200 900
+Wire Wire Line
+	1200 900  2525 900
+Wire Wire Line
+	2525 900  2525 2325
+Connection ~ 2525 2325
+Wire Wire Line
+	1350 1000 1350 900
+Connection ~ 1350 900
 $EndSCHEMATC
